Commit message: 20251021

File: amr_robots_description/urdf/pioneer3dx.urdf.xacro (robot description, xacro)
@@ -47,5 +47,5 @@
   </joint>
   <!-- Top Plate -->
-  <link name="top_plate">
+<!--
     <inertial>
       <mass value="0.01"/>
@@ -66,4 +66,5 @@
    <origin xyz="-0.045 0 0.234" rpy="0 0 0"/>
   </joint>
+-->
   <!-- Front Sonar -->
   <link name="front_sonar">
@@ -131,4 +132,14 @@
         <cylinder radius="${caster_wheel_radius}" length="${caster_wheel_width}"/>
       </geometry>
+      <surface>
+        <friction>
+          <ode>
+            <mu>100000.0</mu>
+            <mu2>100000.0</mu2>
+            <slip1>0.0</slip1>
+            <slip2>0.0</slip2>
+          </ode>
+        </friction>
+      </surface>
     </collision>
   </link>
@@ -139,5 +150,5 @@
     <origin xyz="0 0 0" rpy="${pi/2} ${pi/2} 0"/>
     <axis xyz="0 0 1"/>
-    <limit effort="10" velocity="10"/>
+      <limit effort="10" velocity="10" lower="-1e16" upper="1e16"/>
   </joint>
   <!-- Wheel macro -->
@@ -177,4 +188,14 @@
           <cylinder radius="${wheel_radius}" length="${wheel_width}"/>
         </geometry>
+        <surface>
+          <friction>
+            <ode>
+              <mu>100000.0</mu>
+              <mu2>100000.0</mu2>
+              <slip1>0.0</slip1>
+              <slip2>0.0</slip2>
+            </ode>
+          </friction>
+        </surface>
       </collision>
       <xacro:cylinder_inertia m="1.5" r="${wheel_radius}" h="${wheel_width}"/>
@@ -186,5 +207,5 @@
       <origin xyz="0 0 0" rpy="${pi/2} ${pi/2} 0"/>
       <axis xyz="0 0 1"/>
-      <limit effort="10" velocity="10"/>
+      <limit effort="10" velocity="10" lower="-1e16" upper="1e16"/>
     </joint>
   </xacro:macro>

Commit message: 20251021

File: amr_robots_description/urdf/pioneer3dx.urdf.xacro (robot description, xacro)
@@ -150,5 +150,5 @@
     <origin xyz="0 0 0" rpy="${pi/2} ${pi/2} 0"/>
     <axis xyz="0 0 1"/>
-      <limit effort="10" velocity="10" lower="-1e16" upper="1e16"/>
+    <limit effort="10" velocity="10" lower="-1e16" upper="1e16"/>
   </joint>
   <!-- Wheel macro -->
@@ -205,5 +205,5 @@
       <child link="${prefix}_wheel"/>
       <!--<origin xyz="0 ${y_offset} ${wheel_radius}" rpy="${pi/2} ${pi/2} 0"/>-->
-      <origin xyz="0 0 0" rpy="${pi/2} ${pi/2} 0"/>
+      <origin xyz="0 0 0" rpy="${-pi/2} ${-pi/2} 0"/>
       <axis xyz="0 0 1"/>
       <limit effort="10" velocity="10" lower="-1e16" upper="1e16"/>

Commit message: 20251021

File: amr_robots_description/urdf/pioneer3dx.urdf.xacro (robot description, xacro)
@@ -148,5 +148,5 @@
     <child link="caster_wheel"/>
     <!--<origin xyz="-0.211 0 0.039" rpy="${pi/2} ${pi/2} 0"/>-->
-    <origin xyz="0 0 0" rpy="${pi/2} ${pi/2} 0"/>
+    <origin xyz="-0.025 0 -0.025" rpy="${pi/2} ${pi/2} 0"/>
     <axis xyz="0 0 1"/>
     <limit effort="10" velocity="10" lower="-1e16" upper="1e16"/>
