Commit message: added lidar

File: amr_gazebo/models/robots/pioneer3dx.sdf.xacro (robot description, xacro)
@@ -311,4 +311,42 @@
         filename="libgz-sim-joint-state-publisher-system.so">
       </plugin>
+      <plugin
+        filename="gz-sim-sensors-system"
+        name="gz::sim::systems::Sensors">
+        <render_engine>ogre2</render_engine>
+      </plugin>
+      <frame name="lidar_frame" attached_to='base_link'>
+          <pose>0.0 0 0.25 0 0 0</pose>
+      </frame>
+      <link name="lidar">
+        <sensor name='gpu_lidar' type='gpu_lidar'>"
+          <pose relative_to='base_frame'>0 0 0 0 0 0</pose>
+          <topic>lidar</topic>
+          <update_rate>10</update_rate>
+          <ray>
+              <scan>
+                  <horizontal>
+                      <samples>640</samples>
+                      <resolution>1</resolution>
+                      <min_angle>-1.396263</min_angle>
+                      <max_angle>1.396263</max_angle>
+                  </horizontal>
+                  <vertical>
+                      <samples>1</samples>
+                      <resolution>0.01</resolution>
+                      <min_angle>0</min_angle>
+                      <max_angle>0</max_angle>
+                  </vertical>
+              </scan>
+              <range>
+                  <min>0.08</min>
+                  <max>10.0</max>
+                  <resolution>0.01</resolution>
+              </range>
+          </ray>
+          <always_on>1</always_on>
+          <visualize>true</visualize>
+        </sensor>
+      </link>
     </model>
   </xacro:macro>

File: amr_robots_description/urdf/pioneer3dx.urdf.xacro (robot description, xacro)
@@ -1,4 +1,5 @@
 <?xml version="1.0"?>
 <robot name="pioneer3dx" xmlns:xacro="http://www.ros.org/wiki/xacro">
+  <xacro:include filename="$(find amr_robots_description)/urdf/sensors/rplidar.urdf.xacro" />
   <!-- Define robot constants -->
   <xacro:property name="base_width" value="0.34"/>
@@ -7,4 +8,7 @@
   <xacro:property name="caster_wheel_radius" value="0.0375"/>
   <xacro:property name="caster_wheel_width" value="0.01"/>
+  <xacro:property name="rplidar_x_offset"              value="0"/>
+  <xacro:property name="rplidar_y_offset"              value="0"/>
+  <xacro:property name="rplidar_z_offset"              value="0.25"/>
   <!-- Macro: cylinder inertia -->
   <xacro:macro name="cylinder_inertia" params="m r h">
@@ -47,5 +51,5 @@
   </joint>
   <!-- Top Plate -->
-<!--
+  <link name="top_plate">
     <inertial>
       <mass value="0.01"/>
@@ -66,5 +70,4 @@
    <origin xyz="-0.045 0 0.234" rpy="0 0 0"/>
   </joint>
--->
   <!-- Front Sonar -->
   <link name="front_sonar">
@@ -212,4 +215,8 @@
   <xacro:wheel prefix="left" y_offset="${base_width/2}"/>
   <xacro:wheel prefix="right" y_offset="${-base_width/2}"/>
+  <xacro:rplidar name="rplidar" parent_link="base_link">
+    <origin xyz="${rplidar_x_offset} ${rplidar_y_offset} ${rplidar_z_offset}"
+            rpy="0 0 ${pi/2}"/>
+  </xacro:rplidar>
   <gazebo>
     <!-- DiffDrive Plugin -->
