Commit message: 20251022

File: amr_robots_description/urdf/sensors/rplidar.urdf.xacro (robot description, xacro)
@@ -1,80 +1,44 @@
 <?xml version="1.0"?>
 <robot xmlns:xacro="http://ros.org/wiki/xacro">
-  <xacro:macro name="rplidar" params="name parent_link *origin">
-    <!-- Conversion macros -->
-    <xacro:property name="cm2m"    value="${1/100.0}"/>
-    <xacro:property name="mm2m"    value="${1/1000.0}"/>
-    <xacro:property name="in2m"    value="0.0254"/>
-    <xacro:property name="deg2rad" value="${pi/180.0}"/>
-    <xacro:macro name="inertial_cuboid_with_pose" params="mass x y z *origin">
-      <inertial>
-        <mass value="${mass}" />
-        <xacro:insert_block name="origin"/>
-        <inertia ixx="${(1/12) * mass * (y*y + z*z)}" ixy="0.0" ixz="0.0"
-          iyy="${(1/12) * mass * (x*x + z*z)}" iyz="0.0"
-          izz="${(1/12) * mass * (x*x + y*y)}" />
-      </inertial>
-    </xacro:macro>
-    <xacro:macro name="inertial_cuboid" params="mass x y z">
-      <xacro:inertial_cuboid_with_pose mass="${mass}" x="${x}" y="${y}" z="${z}">
-        <origin xyz="0 0 0" />
-      </xacro:inertial_cuboid_with_pose>
-    </xacro:macro>
-    <xacro:property name="mass"       value="0.17"/>
-    <xacro:property name="length_x"   value="${7.1*cm2m}" />
-    <xacro:property name="length_y"   value="${10*cm2m}" />
-    <xacro:property name="length_z"   value="${6*cm2m}" />
-    <xacro:property name="collision_x_offset" value="${0*cm2m}" />
-    <xacro:property name="collision_y_offset" value="${1.3*cm2m}" />
-    <xacro:property name="collision_z_offset" value="${-1.9*cm2m}" />
-    <joint name="${name}_joint" type="fixed">
-      <parent link="${parent_link}"/>
-      <child link="${name}_link"/>
-      <xacro:insert_block name="origin"/>
-    </joint>
-    <link name="${name}_link">
-      <visual>
-        <geometry>
-          <mesh filename="package://amr_robots_description/meshes/rplidar.dae" scale="1 1 1" />
-        </geometry>
-      </visual>
-      <collision>
-        <origin xyz="${collision_x_offset} ${collision_y_offset} ${collision_z_offset}" rpy="0 0 0"/>
-        <geometry>
-          <box size="${length_x} ${length_y} ${length_z}"/>
-        </geometry>
-      </collision>
-      <xacro:inertial_cuboid mass="${mass}" x="${length_x}" y="${length_y}" z="${length_z}"/>
-      <gazebo reference="${name}_link">
-        <sensor name="lidar" type="ray">
-          <pose>0 0 0.5 0 0 0</pose>
-          <topic>lidar</topic>
-          <update_rate>10</update_rate>
-          <ray>
-            <scan>
-              <horizontal>
-                <samples>640</samples>
-                <resolution>1</resolution>
-                <min_angle>-1.396263</min_angle>
-                <max_angle>1.396263</max_angle>
-              </horizontal>
-              <vertical>
-                <samples>1</samples>
-                <resolution>0.01</resolution>
-                <min_angle>0</min_angle>
-                <max_angle>0</max_angle>
-              </vertical>
-            </scan>
-            <range>
-              <min>0.08</min>
-              <max>10.0</max>
-              <resolution>0.01</resolution>
-            </range>
-          </ray>
-          <always_on>true</always_on>
-          <visualize>true</visualize>
-        </sensor>
-      </gazebo>
-    </link>
-  </xacro:macro>
+<xacro:macro name="rplidar" params="name parent_link *origin">
+  <xacro:include filename="$(find amr_robots_description)/urdf/common_properties/common_properties.urdf.xacro"/>
+  <xacro:property name="mass"       value="0.17"/>
+  <xacro:property name="length_x"   value="${7.1*cm2m}" />
+  <xacro:property name="length_y"   value="${10*cm2m}" />
+  <xacro:property name="length_z"   value="${6*cm2m}" />
+  <xacro:property name="collision_x_offset"       value="${0*cm2m}" />
+  <xacro:property name="collision_y_offset"       value="${1.3*cm2m}" />
+  <xacro:property name="collision_z_offset"       value="${-1.9*cm2m}" />
+  <joint name="${name}_joint" type="fixed">
+    <parent link="${parent_link}"/>
+    <child link="${name}_link"/>
+    <xacro:insert_block name="origin"/>
+  </joint>
+  <link name="${name}_link">
+    <visual>
+      <geometry>
+        <mesh filename="package://amr_robots_description/meshes/rplidar.dae" scale="1 1 1" />
+      </geometry>
+    </visual>
+    <collision>
+      <origin xyz="${collision_x_offset} ${collision_y_offset} ${collision_z_offset}"/>
+      <geometry>
+        <box size="${length_x} ${length_y} ${length_z}"/>
+      </geometry>
+    </collision>
+    <xacro:inertial_cuboid mass="0.17" x="${length_x}" y="${length_y}" z="${length_z}"/>
+  </link>
+  <gazebo reference="${name}_link">
+    <xacro:ray_sensor sensor_name="${name}"
+                  update_rate="62.0" visualize="1"
+                  h_samples="640" h_res="1.0" h_min_angle="${-pi}" h_max_angle="${pi}"
+                  r_min="0.164" r_max="12.0" r_res="0.01">
+                  <plugin name="dummy" filename="dummyfile"></plugin>
+    </xacro:ray_sensor>
+    <xacro:material_darkgray/>
+  </gazebo>
+  <gazebo reference="${name}_joint">
+    <preserveFixedJoint>true</preserveFixedJoint>
+  </gazebo>
+</xacro:macro>
 </robot>
