Commit message: 20251124

File: p3dx_description/urdf/mech/base.urdf.xacro (robot description, xacro)
@@ -21,35 +21,4 @@
     <link name="base_footprint"/>
     <link name="base_link"/>
-<!--
-    <link name="base_link">
-      <visual>
-        <origin xyz="0 0 0" rpy="0 0 0"/>
-        <geometry>
-          <xacro:if value="${mesh_file == ''}">
-            <box size="${length} ${width} ${height}"/>
-          </xacro:if>
-          <xacro:unless value="${mesh_file == ''}">
-            <mesh filename="${mesh_file}" scale="1 1 1"/>
-          </xacro:unless>
-        </geometry>
-        <material name="yellow">
-          <color rgba="0.8784 0.6627 0.6627 1.0"/>
-        </material>
-      </visual>
-      <collision>
-        <origin xyz="0 0 0" rpy="0 0 0"/>
-        <geometry>
-          <box size="${length} ${width} ${height}"/>
-        </geometry>
-      </collision>
-      <inertial>
-        <origin xyz="0 0 0" rpy="0 0 0"/>
-        <mass value="${mass}"/>
-        <inertia ixx="${(1/12) * mass * ((width  * width)  + (height * height))}" ixy="0.0" ixz="0.0"
-                 iyy="${(1/12) * mass * ((length * length) + (height * height))}" iyz="0.0"
-                 izz="${(1/12) * mass * ((length * length) + (width  * width))}"/>
-      </inertial>
-    </link>
--->
     <!-- Chassis -->
     <link name="chassis">
@@ -77,149 +46,89 @@
       <origin xyz="-0.045 0 0.148" rpy="0 0 0"/>
     </joint>
-  <!-- Top Plate -->
-  <link name="top_plate">
-    <inertial>
-      <mass value="0.01"/>
-      <inertia ixx="1" iyy="1" izz="1" ixy="0" ixz="0" iyz="0"/>
-    </inertial>
-    <visual>
-      <geometry>
-        <mesh filename="package://p3dx_description/meshes/p3dx_meshes/top.stl"/>
-      </geometry>
-      <material name="gray">
-        <color rgba="0.038 0.038 0.038 1"/>
-      </material>
-    </visual>
-  </link>
-  <joint name="base_top_joint" type="fixed">
-    <parent link="base_link"/>
-    <child link="top_plate"/>
-   <origin xyz="-0.045 0 0.234" rpy="0 0 0"/>
-  </joint>
-  <!-- Front Sonar -->
-  <link name="front_sonar">
-    <inertial>
-      <mass value="0.0001"/>
-      <inertia ixx="1" iyy="1" izz="1" ixy="0" ixz="0" iyz="0"/>
-    </inertial>
-    <visual>
-      <geometry>
-        <mesh filename="package://p3dx_description/meshes/p3dx_meshes/front_sonar.stl"/>
-      </geometry>
-    </visual>
-  </link>
-  <joint name="base_front_joint" type="fixed">
-    <parent link="base_link"/>
-    <child link="front_sonar"/>
-    <origin xyz="-0.198 0 0.208" rpy="0 0 0"/>
-  </joint>
-  <!-- Back Sonar -->
-  <link name="back_sonar">
-    <inertial>
-      <mass value="0.0001"/>
-      <inertia ixx="1" iyy="1" izz="1" ixy="0" ixz="0" iyz="0"/>
-    </inertial>
-    <visual>
-      <geometry>
-        <mesh filename="package://p3dx_description/meshes/p3dx_meshes/back_sonar.stl"/>
-      </geometry>
-    </visual>
-  </link>
-  <joint name="base_back_joint" type="fixed">
-    <parent link="base_link"/>
-    <child link="back_sonar"/>
-    <origin xyz="0.109 0 0.209" rpy="0 0 0"/>
-  </joint>
-  <link name="caster_swivel">
-    <inertial>
-      <mass value="0.0001"/>
-      <inertia ixx="1" iyy="1" izz="1" ixy="0" ixz="0" iyz="0"/>
-    </inertial>
-    <visual>
-      <geometry>
-        <mesh filename="package://p3dx_description/meshes/p3dx_meshes/caster_swivel.stl"/>
-      </geometry>
-    </visual>
-  </link>
-  <joint name="base_caster_swivel_joint" type="fixed">
-    <parent link="base_link"/>
-    <child link="caster_swivel"/>
-    <origin xyz="-0.185 0 0.055" rpy="0 0 0"/>
-  </joint>
-  <!-- Caster wheel -->
-  <link name="caster_wheel">
-    <inertial>
-      <mass value="0.1"/>
-      <inertia ixx="0.0124" iyy="0.0152" izz="0.0117" ixy="0" ixz="0" iyz="0"/>
-    </inertial>
-    <visual>
-      <geometry>
-        <cylinder radius="${caster_wheel_radius}" length="${caster_wheel_width}"/>
-      </geometry>
-    </visual>
-    <collision>
-      <geometry>
-        <cylinder radius="${caster_wheel_radius}" length="${caster_wheel_width}"/>
-      </geometry>
-      <surface>
-        <friction>
-          <ode>
-            <mu>100000.0</mu>
-            <mu2>100000.0</mu2>
-            <slip1>0.0</slip1>
-            <slip2>0.0</slip2>
-          </ode>
-        </friction>
-      </surface>
-    </collision>
-  </link>
-  <!--<joint name="caster_swivel_hubcap_joint" type="revolute">-->
-  <joint name="caster_swivel_hubcap_joint" type="fixed">
-    <parent link="caster_swivel"/>
-    <child link="caster_wheel"/>
-    <!--<origin xyz="-0.211 0 0.039" rpy="${pi/2} ${pi/2} 0"/>-->
-    <origin xyz="-0.025 0 -0.025" rpy="${pi/2} ${pi/2} 0"/>
-    <axis xyz="0 0 1"/>
-    <limit effort="10" velocity="10" lower="-1e16" upper="1e16"/>
-  </joint>
-  <!-- Wheel macro -->
-  <xacro:macro name="wheel" params="prefix y_offset">
-    <link name="${prefix}_hub">
-      <inertial>
-        <mass value="0.1"/>
-        <inertia ixx="0.01" iyy="0.01" izz="0.01" ixy="0" ixz="0" iyz="0"/>
-      </inertial>
-      <!--
-      <visual>
-        <geometry>
-          <mesh filename="package://p3dx_description/meshes/p3dx_meshes/${prefix}_hubcap.stl"/>
-        </geometry>
-      </visual>
-      -->
-      <xacro:cylinder_inertia m="0.1" r="${wheel_radius-0.05}" h="${wheel_width}"/>
-    </link>
-    <joint name="${prefix}_hub_joint" type="fixed">
-      <parent link="base_link"/>
-      <child link="${prefix}_hub"/>
-      <origin xyz="0 ${y_offset} ${wheel_radius}" rpy="0 0 0"/>
-    </joint>
-    <link name="${prefix}_wheel">
-      <inertial>
-        <mass value="1.5"/>
-        <inertia ixx="0.01" iyy="0.01" izz="0.01" ixy="0" ixz="0" iyz="0"/>
-      </inertial>
-      <visual>
-        <geometry>
-          <cylinder radius="${wheel_radius}" length="${wheel_width}"/>
-        </geometry>
-        <material name="black">
+    <!-- Top Plate -->
+    <link name="top_plate">
+      <inertial>
+        <mass value="0.01"/>
+        <inertia ixx="1" iyy="1" izz="1" ixy="0" ixz="0" iyz="0"/>
+      </inertial>
+      <visual>
+        <geometry>
+          <mesh filename="package://p3dx_description/meshes/p3dx_meshes/top.stl"/>
+        </geometry>
+        <material name="gray">
           <color rgba="0.038 0.038 0.038 1"/>
         </material>
       </visual>
+    </link>
+    <joint name="base_top_joint" type="fixed">
+      <parent link="base_link"/>
+      <child link="top_plate"/>
+    <origin xyz="-0.045 0 0.234" rpy="0 0 0"/>
+    </joint>
+    <!-- Front Sonar -->
+    <link name="front_sonar">
+      <inertial>
+        <mass value="0.0001"/>
+        <inertia ixx="1" iyy="1" izz="1" ixy="0" ixz="0" iyz="0"/>
+      </inertial>
+      <visual>
+        <geometry>
+          <mesh filename="package://p3dx_description/meshes/p3dx_meshes/front_sonar.stl"/>
+        </geometry>
+      </visual>
+    </link>
+    <joint name="base_front_joint" type="fixed">
+      <parent link="base_link"/>
+      <child link="front_sonar"/>
+      <origin xyz="-0.198 0 0.208" rpy="0 0 0"/>
+    </joint>
+    <!-- Back Sonar -->
+    <link name="back_sonar">
+      <inertial>
+        <mass value="0.0001"/>
+        <inertia ixx="1" iyy="1" izz="1" ixy="0" ixz="0" iyz="0"/>
+      </inertial>
+      <visual>
+        <geometry>
+          <mesh filename="package://p3dx_description/meshes/p3dx_meshes/back_sonar.stl"/>
+        </geometry>
+      </visual>
+    </link>
+    <joint name="base_back_joint" type="fixed">
+      <parent link="base_link"/>
+      <child link="back_sonar"/>
+      <origin xyz="0.109 0 0.209" rpy="0 0 0"/>
+    </joint>
+    <link name="caster_swivel">
+      <inertial>
+        <mass value="0.0001"/>
+        <inertia ixx="1" iyy="1" izz="1" ixy="0" ixz="0" iyz="0"/>
+      </inertial>
+      <visual>
+        <geometry>
+          <mesh filename="package://p3dx_description/meshes/p3dx_meshes/caster_swivel.stl"/>
+        </geometry>
+      </visual>
+    </link>
+    <joint name="base_caster_swivel_joint" type="fixed">
+      <parent link="base_link"/>
+      <child link="caster_swivel"/>
+      <origin xyz="-0.185 0 0.055" rpy="0 0 0"/>
+    </joint>
+    <!-- Caster wheel -->
+    <link name="caster_wheel">
+      <inertial>
+        <mass value="0.1"/>
+        <inertia ixx="0.0124" iyy="0.0152" izz="0.0117" ixy="0" ixz="0" iyz="0"/>
+      </inertial>
+      <visual>
+        <geometry>
+          <cylinder radius="${caster_wheel_radius}" length="${caster_wheel_width}"/>
+        </geometry>
+      </visual>
       <collision>
         <geometry>
-          <cylinder radius="${wheel_radius}" length="${wheel_width}"/>
-        </geometry>
-<!--
+          <cylinder radius="${caster_wheel_radius}" length="${caster_wheel_width}"/>
+        </geometry>
         <surface>
           <friction>
@@ -232,19 +141,79 @@
           </friction>
         </surface>
--->
       </collision>
-      <xacro:cylinder_inertia m="1.5" r="${wheel_radius}" h="${wheel_width}"/>
-    </link>
-    <joint name="${prefix}_wheel_joint" type="revolute">
-      <parent link="${prefix}_hub"/>
-      <child link="${prefix}_wheel"/>
-      <!--<origin xyz="0 ${y_offset} ${wheel_radius}" rpy="${pi/2} ${pi/2} 0"/>-->
-      <origin xyz="0 0 0" rpy="${-pi/2} ${-pi/2} 0"/>
+    </link>
+    <!--<joint name="caster_swivel_hubcap_joint" type="revolute">-->
+    <joint name="caster_swivel_hubcap_joint" type="fixed">
+      <parent link="caster_swivel"/>
+      <child link="caster_wheel"/>
+      <!--<origin xyz="-0.211 0 0.039" rpy="${pi/2} ${pi/2} 0"/>-->
+      <origin xyz="-0.025 0 -0.025" rpy="${pi/2} ${pi/2} 0"/>
       <axis xyz="0 0 1"/>
       <limit effort="10" velocity="10" lower="-1e16" upper="1e16"/>
     </joint>
-  </xacro:macro>
-  <xacro:wheel prefix="left" y_offset="${base_width/2}"/>
-  <xacro:wheel prefix="right" y_offset="${-base_width/2}"/>
+    <!-- Wheel macro -->
+    <xacro:macro name="wheel" params="prefix y_offset">
+      <link name="${prefix}_hub">
+        <inertial>
+          <mass value="0.1"/>
+          <inertia ixx="0.01" iyy="0.01" izz="0.01" ixy="0" ixz="0" iyz="0"/>
+        </inertial>
+        <!--
+        <visual>
+          <geometry>
+            <mesh filename="package://p3dx_description/meshes/p3dx_meshes/${prefix}_hubcap.stl"/>
+          </geometry>
+        </visual>
+        -->
+        <xacro:cylinder_inertia m="0.1" r="${wheel_radius-0.05}" h="${wheel_width}"/>
+      </link>
+      <joint name="${prefix}_hub_joint" type="fixed">
+        <parent link="base_link"/>
+        <child link="${prefix}_hub"/>
+        <origin xyz="0 ${y_offset} ${wheel_radius}" rpy="0 0 0"/>
+      </joint>
+      <link name="${prefix}_wheel">
+        <inertial>
+          <mass value="1.5"/>
+          <inertia ixx="0.01" iyy="0.01" izz="0.01" ixy="0" ixz="0" iyz="0"/>
+        </inertial>
+        <visual>
+          <geometry>
+            <cylinder radius="${wheel_radius}" length="${wheel_width}"/>
+          </geometry>
+          <material name="black">
+            <color rgba="0.038 0.038 0.038 1"/>
+          </material>
+        </visual>
+        <collision>
+          <geometry>
+            <cylinder radius="${wheel_radius}" length="${wheel_width}"/>
+          </geometry>
+  <!--
+          <surface>
+            <friction>
+              <ode>
+                <mu>100000.0</mu>
+                <mu2>100000.0</mu2>
+                <slip1>0.0</slip1>
+                <slip2>0.0</slip2>
+              </ode>
+            </friction>
+          </surface>
+  -->
+        </collision>
+        <xacro:cylinder_inertia m="1.5" r="${wheel_radius}" h="${wheel_width}"/>
+      </link>
+      <joint name="${prefix}_wheel_joint" type="revolute">
+        <parent link="${prefix}_hub"/>
+        <child link="${prefix}_wheel"/>
+        <!--<origin xyz="0 ${y_offset} ${wheel_radius}" rpy="${pi/2} ${pi/2} 0"/>-->
+        <origin xyz="0 0 0" rpy="${-pi/2} ${-pi/2} 0"/>
+        <axis xyz="0 0 1"/>
+        <limit effort="10" velocity="10" lower="-1e16" upper="1e16"/>
+      </joint>
+    </xacro:macro>
+    <xacro:wheel prefix="left" y_offset="${base_width/2}"/>
+    <xacro:wheel prefix="right" y_offset="${-base_width/2}"/>
     <joint name="base_to_footprint" type="fixed">
       <parent link="base_footprint"/>

File: p3dx_description/urdf/p3dx.urdf.xacro (robot description, xacro)
@@ -55,37 +55,4 @@
     mesh_file="${base_mesh_file}"
   />
-<!--
-  <xacro:wheel
-    side="left"
-    radius="${wheel_radius}"
-    width="${wheel_width}"
-    pos_x="${wheel_pos_x}"
-    pos_y="${base_width/2}"
-    pos_z="${wheel_radius}"
-    mass="${wheel_mass}"
-    mesh_file="${wheel_mesh_file}"
-  />
-  <xacro:wheel
-    side="right"
-    radius="${wheel_radius}"
-    width="${wheel_width}"
-    pos_x="${wheel_pos_x}"
-    pos_y="${-base_width/2}"
-    pos_z="${wheel_radius}"
-    mass="${wheel_mass}"
-    mesh_file="${wheel_mesh_file}"
-  />
--->
-<!--
-  <xacro:if value="${rear_caster_wheel}">
-    <xacro:caster_wheel
-      side="rear"
-      mass="0.01"
-      base_length="${base_length}"
-      wheel_radius="${caster_wheel_radius}"
-      wheel_pos_z="${wheel_pos_z}"
-    />
-  </xacro:if>
--->
   <xacro:imu/>
   <xacro:rplidar frame_id="laser" parent_link="base_link">
@@ -103,9 +70,3 @@
   </xacro:depth_sensor>
 -->
-<!--
-  <xacro:diff_drive_controller
-    wheel_separation="${wheel_pos_y * 2}"
-    wheel_radius="${wheel_radius}"
-  />
--->
 </robot>
