File: kiCad/P3DX_Controller/P3DX_Controller.kicad_sch (KiCad schematic)
At the start: 1 part, among them U1 ESP32-WROOM-32E

Commit message: 20251110
Parts:
- added U2: ~, railtrack:1.77 LCD Display 128x160, symbol railtrack:1.77_LCD_Display
Changed lines of the file:
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@@
+		)
+	)
+	(symbol
+		(lib_id "railtrack:1.77_LCD_Display")
+		(at 125.73 58.42 0)
+		(unit 1)
+		(exclude_from_sim no)
+		(in_bom yes)
+		(on_board yes)
+		(dnp no)
+		(fields_autoplaced yes)
+		(property "Reference" "U2"
+			(at 139.7 62.4811 0)
+			(effects
+				(font
+					(size 1.27 1.27)
+				)
+				(justify left)
+			)
+		)
+		(property "Value" "~"
+			(at 139.7 65.0211 0)
+			(effects
+				(font
+					(size 1.27 1.27)
+				)
+				(justify left)
+			)
+		)
+		(property "Footprint" "railtrack:1.77 LCD Display 128x160"
+			(at 125.73 58.42 0)
+			(effects
+				(font
+					(size 1.27 1.27)
+				)
+				(hide yes)
+			)
+		)
+		(property "Datasheet" ""
+			(at 125.73 58.42 0)
+			(effects
+				(font
+					(size 1.27 1.27)
+				)
+				(hide yes)
+			)
+		)
+		(property "Description" ""
+			(at 125.73 58.42 0)
+			(effects
+				(font
+					(size 1.27 1.27)
+				)
+				(hide yes)
+			)
+		)
+		(pin "3"
+		)
+		(pin "8"
+		)
+		(pin "2"
+		)
+		(pin "7"
+		)
+		(pin "5"
+		)
+		(pin "6"
+		)
+		(pin "1"
+		)
+		(pin "4"
+		)
+		(instances
+			(project ""
+				(path "/ef99843a-7c8a-41b3-bbe8-92aaa291095d"
+					(reference "U2")
+					(unit 1)
+				)
+			)
 		)
 	)

Commit message: 20251118
Parts:
- removed U1: ESP32-WROOM-32E, RF_Module:ESP32-WROOM-32D, symbol RF_Module:ESP32-WROOM-32E
- added J1, J2: Conn_01x10_Pin, Connector_IDC:IDC-Header_2x05_P2.54mm_Vertical, symbol Connector:Conn_01x10_Pin
- added J3: Conn_01x26_Pin, Connector_IDC:IDC-Header_2x13_P2.54mm_Vertical, symbol Connector:Conn_01x26_Pin
- added J5: Conn_01x16_Pin, Connector_IDC:IDC-Header_2x08_P2.54mm_Vertical, symbol Connector:Conn_01x16_Pin
- added U1: ESP32-DevKitC, PCM_Espressif:ESP32-DevKitC, symbol PCM_Espressif:ESP32-DevKitC
Connections:
- new net: U1.14 (GND), U1.32 (GND), U1.38 (GND)

Commit message: linorobot inspiratie
Parts:
- added J4: Conn_01x03_Pin, Connector_PinHeader_1.27mm:PinHeader_1x03_P1.27mm_Vertical, symbol Connector:Conn_01x03_Pin
- added J6: Conn_01x05_Pin, Connector_PinSocket_2.54mm:PinSocket_1x05_P2.54mm_Vertical, symbol Connector:Conn_01x05_Pin
- added U3: TXS0108EPW, railtrack:Texas_TXS0108E_Level_Shifter_Module, symbol Logic_LevelTranslator:TXS0108EPW

Commit message: 20251123
Connections:
- net L_MOTOR_PWM: now reaches J3.1 (Pin_1)
- net L_MOTOR_DIR: now reaches J3.2 (Pin_2)
- net V_BATTERY: now reaches J3.22 (Pin_22)
- net GND: now reaches J3.23 (Pin_23)
- net GND: now also J3.25 (Pin_25), U2.1 (GND), U3.11 (GND)
- net R_MOTOR_PWM: now reaches J3.3 (Pin_3)
- net R_MOTOR_DIR: now reaches J3.4 (Pin_4)
- net MOTOR_ENABLE: now reaches J3.5 (Pin_5)
- net L_ENCODER_A: now reaches J3.6 (Pin_6)
- net L_ENCODER_A: now also U3.20 (B1)
- net R_ENCODER_A: now reaches J3.7 (Pin_7)
- net R_ENCODER_A: now also U3.18 (B2)
- net R_ENCODER_B: now reaches J3.8 (Pin_8)
- net R_ENCODER_B: now also U3.17 (B3)
- net L_ENCODER_B: now reaches J3.9 (Pin_9)
- net L_ENCODER_B: now also U3.16 (B4)
- net +3V3: now reaches U2.2 (VCC)
- net +3V3: now also U3.10 (OE), U3.2 (VCCA)
- net L_ENCODER_A_LV: now reaches U3.1 (A1)
- net VCC: now reaches U3.19 (VCCB)
- net VCC: now also U1.19 (5V)
- net R_ENCODER_A_LV: now reaches U3.3 (A2)
- net R_ENCODER_B_LV: now reaches U3.4 (A3)
- net L_ENCODER_B_LV: now reaches U3.5 (A4)

Commit message: 20251127
Parts:
- added R1, R2: 10k, Resistor_THT:R_Box_L13.0mm_W4.0mm_P9.00mm, symbol Device:R
Connections:
- net +3V3: now also U1.1 (3V3), U2.8 (LED_A)
- net GND: now also J4.2 (Pin_2), J6.4 (Pin_4), U1.14 (GND), U1.32 (GND), U1.38 (GND), R2.2
- net VCC: now also J4.1 (Pin_1), J6.1 (Pin_1)
- net V_BATTERY: now also R1.1
- net lidar-tx: now reaches J6.2 (Pin_2)
- net lidar-tx: now also U1.27 (GPIO16)
- net lidar-rx: now reaches J6.3 (Pin_3)
- net lidar-rx: now also U1.28 (GPIO17)
- net lidar-motor: now reaches J6.5 (Pin_5)
- net display_clk: now reaches U2.3 (SCL)
- net display_clk: now also U1.30 (GPIO18)
- net display_sda: now reaches U2.4 (SDA)
- net display_sda: now also U1.37 (GPIO23)
- net display_rst: now reaches U2.5 (RES)
- net display_rst: now also U1.15 (MTCK/GPIO13/ADC2_CH4)
- net display_RS_DC: now reaches U2.6 (RS)
- net display_RS_DC: now also U1.13 (MTDI/GPIO12/ADC2_CH5)
- net display_cs: now reaches U2.7 (CS)
- net display_cs: now also U1.29 (GPIO5)
- net display_not_used: now reaches U1.31 (GPIO19)
- net i2c-sda: now reaches U1.33 (GPIO21)
- net i2c-scl: now reaches U1.36 (GPIO22)
- net V_BATTERY_MEASUREMENT: now reaches U1.5 (VDET_1/GPIO34/ADC1_CH6)
- net V_BATTERY_MEASUREMENT: now also R1.2, R2.1
Other:
- note added: "#define DISPLAY_CS_PIN 5 #define DISPLAY_RS_DC_PIN 12 #define DISPLAY_RST_PIN 13 #define DISPLAY_CLK_PIN 18 #define DISPLAY_SDA_PIN 23 #define DISPLAY_MISO_PIN 19 // Not used #define RPLIDAR_COM_PORT 2 #define RPLIDAR_TX_PIN 16//35// Never use pin 10 !!!! // Lidar side #define RPLIDAR_RX_PIN 17// 9 // Lidar side #define RPLIDAR_MOTOR_PIN 25 // optioneel: PWM of GPIO voor motor aan/uit"
- moved on the sheet: J5, J6, U1, U2

Commit message: 20251128
Parts:
- added R2: DO NOT PLACE, Resistor_THT:R_Box_L13.0mm_W4.0mm_P9.00mm, symbol Device:R
- J5: renamed from J4; footprint Connector_PinHeader_1.27mm:PinHeader_1x03_P1.27mm_Vertical -> Connector_PinHeader_2.54mm:PinHeader_1x03_P2.54mm_Vertical
- renumbered J3 to J2, J2 to J3, J5 to J4, R2 to R3, U3 to U1, U1 to U3
Connections:
- net V_BATTERY is gone; now on net GND: J2.22 (Pin_22), R1.1
- net GND: now also J1.10 (Pin_10), J1.9 (Pin_9), J3.10 (Pin_10), J3.9 (Pin_9), J4.12 (Pin_12), J4.13 (Pin_13)
- net L_ENCODER_A_LV: now also U3.17 (SD_DATA3/GPIO10)
- net L_ENCODER_B_LV: now also U3.21 (SD_DATA0/GPIO7)
- net L_MOTOR_DIR: now also U3.10 (DAC_2/ADC2_CH9/GPIO26)
- net L_MOTOR_PWM: now also U3.9 (DAC_1/ADC2_CH8/GPIO25)
- net MOTOR_ENABLE: now also U3.26 (ADC2_CH0/GPIO4)
- net R_ENCODER_A_LV: now also U3.16 (SD_DATA2/GPIO9)
- net R_ENCODER_B_LV: now also U3.22 (SD_DATA1/GPIO8)
- net R_MOTOR_DIR: now also U3.20 (SD_CLK/GPIO6)
- net R_MOTOR_PWM: now also U3.11 (ADC2_CH7/GPIO27)
- net VCC: now also J4.1 (Pin_1), J4.2 (Pin_2), R2.1
- net ucp_status: now reaches J4.10 (Pin_10)
- net ucp_status: now also U1.12 (B8)
- net ucp_reset: now reaches J4.3 (Pin_3)
- net ucp_reset: now also U1.15 (B5)
- net ucp_motors: now reaches J4.4 (Pin_4)
- net ucp_motors: now also U1.14 (B6), R2.2
- net ucp_buzzer_pwm: now reaches J4.8 (Pin_8)
- net ucp_buzzer_pwm: now also U1.13 (B7)
- net ucp_power_led: now reaches J4.9 (Pin_9)
- net ucp_reset_lv: now reaches U1.6 (A5)
- net ucp_reset_lv: now also U3.6 (VDET_2/GPIO35/ADC1_CH7)
- net ucp_motors_lv: now reaches U1.7 (A6)
- net ucp_motors_lv: now also U3.3 (SENSOR_VP/GPIO36/ADC1_CH0)
- net ucp_buzzer_pwm_lv: now reaches U1.8 (A7)
- net ucp_buzzer_pwm_lv: now also U3.4 (SENSOR_VN/GPIO39/ADC1_CH3)
- net ucp_status_lv: now reaches U1.9 (A8)
- net ucp_status_lv: now also U3.23 (MTDO/GPIO15/ADC2_CH3)
Other:
- moved on the sheet: J1, J2, J3

Commit message: 20251128
Parts:
- added R4, R5: DO NOT PLACE, Resistor_THT:R_Axial_DIN0204_L3.6mm_D1.6mm_P7.62mm_Horizontal, symbol Device:R
- added U4: ~, p3dx:GY_271, symbol p3dx:GY_271
- J6: footprint Connector_PinSocket_2.54mm:PinSocket_1x05_P2.54mm_Vertical -> Connector_PinHeader_2.54mm:PinHeader_1x05_P2.54mm_Vertical
- R1, R2, R3: footprint Resistor_THT:R_Box_L13.0mm_W4.0mm_P9.00mm -> Resistor_THT:R_Axial_DIN0204_L3.6mm_D1.6mm_P7.62mm_Horizontal
Connections:
- net +3V3: now also R4.1, R5.1, U4.1 (VCC)
- net GND: now also U4.2 (GND)
- net i2c-scl: now also U4.3 (SCL)
- net i2c-sda: now also U4.4 (SDA)
- net front_bumper: now reaches J1.1 (Pin_1)
- net front_bumper: now also J1.2 (Pin_2), J1.3 (Pin_3), J1.4 (Pin_4), J1.5 (Pin_5), J1.6 (Pin_6), J1.7 (Pin_7), J1.8 (Pin_8), U3.7 (32K_XP/GPIO32/ADC1_CH4), R4.2
- net rear_bumper: now reaches J3.1 (Pin_1)
- net rear_bumper: now also J3.2 (Pin_2), J3.3 (Pin_3), J3.4 (Pin_4), J3.5 (Pin_5), J3.6 (Pin_6), J3.7 (Pin_7), J3.8 (Pin_8), U3.8 (32K_XN/GPIO33/ADC1_CH5), R5.2
- net imu_drdy: now reaches U3.12 (MTMS/GPIO14/ADC2_CH6)
- net imu_drdy: now also U4.5 (DRDY)

Commit message: 20251129
Parts:
- removed U4: ~, p3dx:GY_271, symbol p3dx:GY_271
- added C3, C4: 100nF, Capacitor_THT:C_Axial_L3.8mm_D2.6mm_P7.50mm_Horizontal, symbol Device:C
- added CP1, CP2: 100uF/10V, Capacitor_THT:CP_Radial_D5.0mm_P2.50mm, symbol Device:C_Polarized
- added U4: ~, p3dx:MPU6050, symbol p3dx:MPU6050
Connections:
- net +3V3: now also C3.1, CP1.1, U4.1 (Vcc)
- net GND: now also C3.2, C4.2, CP1.2, CP2.2, U4.2 (GND), U4.7 (AD0)
- net VCC: now also C4.1, CP2.1
- net i2c-scl: now also U4.3 (SCL)
- net i2c-sda: now also U4.4 (SDA)
- net imu_drdy renamed imu_int
- net imu_int: now also U4.8 (INTx)
