File: kiCad/P3DX_Controller/P3DX_Controller.kicad_sch (KiCad schematic)
At the start: 20 parts, among them J1 Conn_01x10_Pin, J2 Conn_01x26_Pin, J3 Conn_01x10_Pin, J4 Conn_01x16_Pin, J5 Conn_01x03_Pin, J6 Conn_01x05_Pin, U2 TXS0108EPW, U3 ESP32-S3-DevKitC

Commit message: added buzzer
Parts:
- R2: value 10k -> 560k
- R3: value 10k -> 100k
Connections:
- net front_bumper: now also J3.1 (Pin_1), J3.2 (Pin_2), J3.3 (Pin_3), J3.4 (Pin_4), J3.5 (Pin_5), J3.6 (Pin_6), J3.7 (Pin_7), J3.8 (Pin_8), U3.30 (GPIO45); no longer J1.1 (Pin_1), J1.2 (Pin_2), J1.3 (Pin_3), J1.4 (Pin_4), J1.5 (Pin_5), J1.6 (Pin_6), J1.7 (Pin_7), J1.8 (Pin_8), U3.14 (GPIO46)
- net rear_bumper: now also J1.1 (Pin_1), J1.2 (Pin_2), J1.3 (Pin_3), J1.4 (Pin_4), J1.5 (Pin_5), J1.6 (Pin_6), J1.7 (Pin_7), J1.8 (Pin_8), U3.14 (GPIO46); no longer J3.1 (Pin_1), J3.2 (Pin_2), J3.3 (Pin_3), J3.4 (Pin_4), J3.5 (Pin_5), J3.6 (Pin_6), J3.7 (Pin_7), J3.8 (Pin_8), U3.30 (GPIO45)
Changed lines of the file:
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@@
-		)
-	)
-	(label "rear_bumper"
-		(at 101.6 101.6 0)
-		(effects
-			(font
-				(size 1.27 1.27)
-			)
-			(justify left bottom)
 		)
 	)
@@
 		)
 	)
-	(label "rear_bumper"
+	(label "front_bumper"
 		(at 209.55 54.61 0)
 		(effects
@@
 		)
 	)
-	(label "front_bumper"
+	(label "rear_bumper"
 		(at 182.88 54.61 0)
 		(effects
@@
 		)
 	)
+	(label "front_bumper"
+		(at 101.6 101.6 0)
+		(effects
+			(font
+				(size 1.27 1.27)
+			)
+			(justify left bottom)
+		)
+	)
 	(label "V_BATTERY"
 		(at 149.86 106.68 0)
@@
 		)
 	)
-	(label "front_bumper"
+	(label "rear_bumper"
 		(at 101.6 104.14 0)
 		(effects
@@
 			)
 		)
-		(property "Value" "10k"
+		(property "Value" "100k"
 			(at 67.31 182.8799 0)
 			(effects
@@
 			)
 		)
-		(property "Value" "10k"
+		(property "Value" "560k"
 			(at 67.31 175.2599 0)
 			(effects
