File: kiCad/P3DX_Controller/P3DX_Controller.kicad_pcb (KiCad board)
At the start: 2 copper layers, 2 parts, among them U1 ESP32-WROOM-32E

Commit message: 20251118
Parts:
- added J1: Conn_01x10_Pin, Connector_IDC:IDC-Header_2x05_P2.54mm_Vertical, F.Cu at (68.0, 57.1)
- added J2: Conn_01x10_Pin, Connector_IDC:IDC-Header_2x05_P2.54mm_Vertical, F.Cu at (136.6, 57.6)
- added J3: Conn_01x26_Pin, Connector_IDC:IDC-Header_2x13_P2.54mm_Vertical, F.Cu at (92.2, 57.4)
- added J5: Conn_01x16_Pin, Connector_IDC:IDC-Header_2x08_P2.54mm_Vertical, F.Cu at (60.0, 74.9)
- added REF**: MountingHole_3.2mm_M3, MountingHole:MountingHole_3.2mm_M3, F.Cu at (55.0, 55.0)
- added REF**: MountingHole_3.2mm_M3, MountingHole:MountingHole_3.2mm_M3, F.Cu at (55.0, 125.0)
- added REF**: MountingHole_3.2mm_M3, MountingHole:MountingHole_3.2mm_M3, F.Cu at (170.0, 55.0)
- added REF**: MountingHole_3.2mm_M3, MountingHole:MountingHole_3.2mm_M3, F.Cu at (170.0, 125.0)
- U1: value ESP32-WROOM-32E -> ESP32-DevKitC; footprint RF_Module:ESP32-WROOM-32D -> PCM_Espressif:ESP32-DevKitC
- moved U2 55.3 mm to (130.3, 97.5), turned to 90 degrees
- moved U1 34.8 mm to (77.2, 75.9)
Connections:
- U1 pad 1: Net-(U1-GND-Pad1) -> unconnected-(U1-3V3-Pad1)
- U1 pad 14: unconnected-(U1-IO12-Pad14) -> Net-(U1-GND-Pad14)
- U1 pad 15: Net-(U1-GND-Pad1) -> unconnected-(U1-MTCK/GPIO13/ADC2_CH4-Pad15)
- U1 pad 32: unconnected-(U1-NC-Pad32) -> Net-(U1-GND-Pad14)
- U1 pad 38: Net-(U1-GND-Pad1) -> Net-(U1-GND-Pad14)
Other:
- board outline added: 125 x 80 mm

Commit message: linorobot inspiratie
Parts:
- added J4: Conn_01x03_Pin, Connector_PinHeader_1.27mm:PinHeader_1x03_P1.27mm_Vertical, F.Cu at (164.3, 79.2)
- added J6: Conn_01x05_Pin, Connector_PinSocket_2.54mm:PinSocket_1x05_P2.54mm_Vertical, F.Cu at (160.0, 79.8)
- added U3: TXS0108EPW, railtrack:Texas_TXS0108E_Level_Shifter_Module, F.Cu at (202.3, 74.7)

Commit message: 20251123
Parts:
- moved J3 27.9 mm to (120.0, 55.0), turned to -90 degrees
- moved J5 17.6 mm to (60.0, 92.5), turned to 180 degrees
- turned J1 to -90 degrees
- turned J2 to -90 degrees
Connections:
- J3 pad 1: unconnected-(J3-Pin_1-Pad1) -> /L_MOTOR_PWM
- J3 pad 2: unconnected-(J3-Pin_2-Pad2) -> /L_MOTOR_DIR
- J3 pad 22: unconnected-(J3-Pin_22-Pad22) -> /V_BATTERY
- J3 pad 23: unconnected-(J3-Pin_23-Pad23) -> GND
- J3 pad 25: unconnected-(J3-Pin_25-Pad25) -> GND
- J3 pad 3: unconnected-(J3-Pin_3-Pad3) -> /R_MOTOR_PWM
- J3 pad 4: unconnected-(J3-Pin_4-Pad4) -> /R_MOTOR_DIR
- J3 pad 5: unconnected-(J3-Pin_5-Pad5) -> /MOTOR_ENABLE
- J3 pad 6: unconnected-(J3-Pin_6-Pad6) -> /L_ENCODER_A
- J3 pad 7: unconnected-(J3-Pin_7-Pad7) -> /R_ENCODER_A
- J3 pad 8: unconnected-(J3-Pin_8-Pad8) -> /R_ENCODER_B
- J3 pad 9: unconnected-(J3-Pin_9-Pad9) -> /L_ENCODER_B
- U1 pad 1: unconnected-(U1-3V3-Pad1) -> +3V3
- U1 pad 14: Net-(U1-GND-Pad14) -> GND
- U1 pad 19: unconnected-(U1-5V-Pad19) -> VCC
- U1 pad 32: Net-(U1-GND-Pad14) -> GND
- U1 pad 38: Net-(U1-GND-Pad14) -> GND
- U2 pad 1: unconnected-(U2-GND-Pad1) -> GND
- U2 pad 2: unconnected-(U2-VCC-Pad2) -> +3V3
- U3 pad 11: unconnected-(U3-GND-Pad11) -> GND
- U3 pad 16: unconnected-(U3-B4-Pad16) -> /L_ENCODER_B
- U3 pad 17: unconnected-(U3-B3-Pad17) -> /R_ENCODER_B
- U3 pad 18: unconnected-(U3-B2-Pad18) -> /R_ENCODER_A
- U3 pad 19: unconnected-(U3-VCCB-Pad19) -> VCC
- U3 pad 2: unconnected-(U3-VCCA-Pad2) -> +3V3
- U3 pad 20: unconnected-(U3-B1-Pad20) -> /L_ENCODER_A

Commit message: 20251127
Parts:
- added R1: 10k, Resistor_THT:R_Box_L13.0mm_W4.0mm_P9.00mm, F.Cu at (60.0, 105.0)
- added R2: 10k, Resistor_THT:R_Box_L13.0mm_W4.0mm_P9.00mm, F.Cu at (61.0, 115.0)
- moved U3 127.3 mm to (75.0, 74.8)
- moved J4 90.2 mm to (79.3, 109.3)
- moved J6 90.2 mm to (75.0, 110.0)
- moved U1 58.7 mm to (109.4, 125.0), turned to 90 degrees
- moved U2 17.5 mm to (130.0, 80.0), turned to 0 degrees
- moved J2 8.79 mm to (145.0, 55.0)
- moved J1 7.28 mm to (75.0, 55.0)
Connections:
- J4 pad 1: unconnected-(J4-Pin_1-Pad1) -> VCC
- J4 pad 2: unconnected-(J4-Pin_2-Pad2) -> GND
- J6 pad 1: unconnected-(J6-Pin_1-Pad1) -> VCC
- J6 pad 2: unconnected-(J6-Pin_2-Pad2) -> /lidar-tx
- J6 pad 3: unconnected-(J6-Pin_3-Pad3) -> /lidar-rx
- J6 pad 4: unconnected-(J6-Pin_4-Pad4) -> GND
- J6 pad 5: unconnected-(J6-Pin_5-Pad5) -> /lidar-motor
- U1 pad 13: unconnected-(U1-MTDI/GPIO12/ADC2_CH5-Pad13) -> /display_RS_DC
- U1 pad 15: unconnected-(U1-MTCK/GPIO13/ADC2_CH4-Pad15) -> /display_rst
- U1 pad 27: unconnected-(U1-GPIO16-Pad27) -> /lidar-tx
- U1 pad 28: unconnected-(U1-GPIO17-Pad28) -> /lidar-rx
- U1 pad 29: unconnected-(U1-GPIO5-Pad29) -> /display_cs
- U1 pad 30: unconnected-(U1-GPIO18-Pad30) -> /display_clk
- U1 pad 31: unconnected-(U1-GPIO19-Pad31) -> /display_not_used
- U1 pad 33: unconnected-(U1-GPIO21-Pad33) -> /i2c-sda
- U1 pad 36: unconnected-(U1-GPIO22-Pad36) -> /i2c-scl
- U1 pad 37: unconnected-(U1-GPIO23-Pad37) -> /display_sda
- U1 pad 5: unconnected-(U1-VDET_1/GPIO34/ADC1_CH6-Pad5) -> /V_BATTERY_MEASUREMENT
- U2 pad 3: unconnected-(U2-SCL-Pad3) -> /display_clk
- U2 pad 4: unconnected-(U2-SDA-Pad4) -> /display_sda
- U2 pad 5: unconnected-(U2-RES-Pad5) -> /display_rst
- U2 pad 6: unconnected-(U2-RS-Pad6) -> /display_RS_DC
- U2 pad 7: unconnected-(U2-CS-Pad7) -> /display_cs
- U2 pad 8: unconnected-(U2-LED_A-Pad8) -> +3V3
- U3 pad 1: unconnected-(U3-A1-Pad1) -> /L_ENCODER_A_LV
- U3 pad 10: unconnected-(U3-OE-Pad10) -> +3V3
- U3 pad 3: unconnected-(U3-A2-Pad3) -> /R_ENCODER_A_LV
- U3 pad 4: unconnected-(U3-A3-Pad4) -> /R_ENCODER_B_LV
- U3 pad 5: unconnected-(U3-A4-Pad5) -> /L_ENCODER_B_LV

Commit message: 20251128
Parts:
- added R2: DO NOT PLACE, Resistor_THT:R_Box_L13.0mm_W4.0mm_P9.00mm, F.Cu at (81.0, 105.0)
- J5: renamed from J4; footprint Connector_PinHeader_1.27mm:PinHeader_1x03_P1.27mm_Vertical -> Connector_PinHeader_2.54mm:PinHeader_1x03_P2.54mm_Vertical
- renumbered REF** to HOLE1, REF** to HOLE2, REF** to HOLE3, REF** to HOLE4, J3 to J2, J2 to J3, J5 to J4, R2 to R3, U3 to U1, U1 to U3
Connections:
- J1 pad 10: unconnected-(J1-Pin_10-Pad10) -> GND
- J1 pad 9: unconnected-(J1-Pin_9-Pad9) -> GND
- J2 pad 22: /V_BATTERY -> GND
- J3 pad 10: unconnected-(J2-Pin_10-Pad10) -> GND
- J3 pad 9: unconnected-(J2-Pin_9-Pad9) -> GND
- J4 pad 1: unconnected-(J5-Pin_1-Pad1) -> VCC
- J4 pad 10: unconnected-(J5-Pin_10-Pad10) -> /ucp_status
- J4 pad 12: unconnected-(J5-Pin_12-Pad12) -> GND
- J4 pad 13: unconnected-(J5-Pin_13-Pad13) -> GND
- J4 pad 2: unconnected-(J5-Pin_2-Pad2) -> VCC
- J4 pad 3: unconnected-(J5-Pin_3-Pad3) -> /ucp_reset
- J4 pad 4: unconnected-(J5-Pin_4-Pad4) -> /ucp_motors
- J4 pad 8: unconnected-(J5-Pin_8-Pad8) -> /ucp_buzzer_pwm
- J4 pad 9: unconnected-(J5-Pin_9-Pad9) -> /ucp_power_led
- R1 pad 1: /V_BATTERY -> GND
- U1 pad 12: unconnected-(U3-B8-Pad12) -> /ucp_status
- U1 pad 13: unconnected-(U3-B7-Pad13) -> /ucp_buzzer_pwm
- U1 pad 14: unconnected-(U3-B6-Pad14) -> /ucp_motors
- U1 pad 15: unconnected-(U3-B5-Pad15) -> /ucp_reset
- U1 pad 6: unconnected-(U3-A5-Pad6) -> /ucp_reset_lv
- U1 pad 7: unconnected-(U3-A6-Pad7) -> /ucp_motors_lv
- U1 pad 8: unconnected-(U3-A7-Pad8) -> /ucp_buzzer_pwm_lv
- U1 pad 9: unconnected-(U3-A8-Pad9) -> /ucp_status_lv
- U3 pad 10: unconnected-(U1-DAC_2/ADC2_CH9/GPIO26-Pad10) -> /L_MOTOR_DIR
- U3 pad 11: unconnected-(U1-ADC2_CH7/GPIO27-Pad11) -> /R_MOTOR_PWM
- U3 pad 16: unconnected-(U1-SD_DATA2/GPIO9-Pad16) -> /R_ENCODER_A_LV
- U3 pad 17: unconnected-(U1-SD_DATA3/GPIO10-Pad17) -> /L_ENCODER_A_LV
- U3 pad 20: unconnected-(U1-SD_CLK/GPIO6-Pad20) -> /R_MOTOR_DIR
- U3 pad 21: unconnected-(U1-SD_DATA0/GPIO7-Pad21) -> /L_ENCODER_B_LV
- U3 pad 22: unconnected-(U1-SD_DATA1/GPIO8-Pad22) -> /R_ENCODER_B_LV
- U3 pad 23: unconnected-(U1-MTDO/GPIO15/ADC2_CH3-Pad23) -> /ucp_status_lv
- U3 pad 26: unconnected-(U1-ADC2_CH0/GPIO4-Pad26) -> /MOTOR_ENABLE
- U3 pad 3: unconnected-(U1-SENSOR_VP/GPIO36/ADC1_CH0-Pad3) -> /ucp_motors_lv
- U3 pad 4: unconnected-(U1-SENSOR_VN/GPIO39/ADC1_CH3-Pad4) -> /ucp_buzzer_pwm_lv
- U3 pad 6: unconnected-(U1-VDET_2/GPIO35/ADC1_CH7-Pad6) -> /ucp_reset_lv
- U3 pad 9: unconnected-(U1-DAC_1/ADC2_CH8/GPIO25-Pad9) -> /L_MOTOR_PWM
Routing:
- net VCC: track 0.00 -> 155.7 mm, vias 0 -> 1
- net /L_ENCODER_A_LV: track 0.00 -> 124.0 mm, vias 0 -> 1
- net /R_ENCODER_A_LV: track 0.00 -> 115.4 mm, vias 0 -> 1
- net +3V3: track 0.00 -> 110.9 mm
- net /R_ENCODER_B_LV: track 0.00 -> 93.2 mm, vias 0 -> 1
- net /L_ENCODER_B_LV: track 0.00 -> 85.5 mm
- net /display_rst: track 0.00 -> 84.3 mm, vias 0 -> 1
- net /ucp_reset_lv: track 0.00 -> 84.1 mm, vias 0 -> 1
- net /display_RS_DC: track 0.00 -> 81.6 mm, vias 0 -> 1
- net /R_MOTOR_PWM: track 0.00 -> 80.9 mm
- net /R_MOTOR_DIR: track 0.00 -> 77.9 mm, vias 0 -> 1
- net /V_BATTERY_MEASUREMENT: track 0.00 -> 76.8 mm
- net /ucp_status_lv: track 0.00 -> 76.2 mm
- net /L_MOTOR_PWM: track 0.00 -> 75.0 mm
- net /ucp_motors_lv: track 0.00 -> 73.8 mm, vias 0 -> 1
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- added copper zone on B.Cu, net GND
- added copper zone on F.Cu, net GND

Commit message: 20251128
Parts:
- added R4: DO NOT PLACE, Resistor_THT:R_Axial_DIN0204_L3.6mm_D1.6mm_P7.62mm_Horizontal, F.Cu at (88.0, 113.0)
- added R5: DO NOT PLACE, Resistor_THT:R_Axial_DIN0204_L3.6mm_D1.6mm_P7.62mm_Horizontal, F.Cu at (88.0, 121.0)
- added U4: ~, p3dx:GY_271, F.Cu at (166.1, 93.9)
- J6: footprint Connector_PinSocket_2.54mm:PinSocket_1x05_P2.54mm_Vertical -> Connector_PinHeader_2.54mm:PinHeader_1x05_P2.54mm_Vertical
- R1, R2, R3: footprint Resistor_THT:R_Box_L13.0mm_W4.0mm_P9.00mm -> Resistor_THT:R_Axial_DIN0204_L3.6mm_D1.6mm_P7.62mm_Horizontal
Connections:
- J1 pad 1: unconnected-(J1-Pin_1-Pad1) -> /front_bumper
- J1 pad 2: unconnected-(J1-Pin_2-Pad2) -> /front_bumper
- J1 pad 3: unconnected-(J1-Pin_3-Pad3) -> /front_bumper
- J1 pad 4: unconnected-(J1-Pin_4-Pad4) -> /front_bumper
- J1 pad 5: unconnected-(J1-Pin_5-Pad5) -> /front_bumper
- J1 pad 6: unconnected-(J1-Pin_6-Pad6) -> /front_bumper
- J1 pad 7: unconnected-(J1-Pin_7-Pad7) -> /front_bumper
- J1 pad 8: unconnected-(J1-Pin_8-Pad8) -> /front_bumper
- J3 pad 1: unconnected-(J2-Pin_1-Pad1) -> /rear_bumper
- J3 pad 2: unconnected-(J2-Pin_2-Pad2) -> /rear_bumper
- J3 pad 3: unconnected-(J2-Pin_3-Pad3) -> /rear_bumper
- J3 pad 4: unconnected-(J2-Pin_4-Pad4) -> /rear_bumper
- J3 pad 5: unconnected-(J2-Pin_5-Pad5) -> /rear_bumper
- J3 pad 6: unconnected-(J2-Pin_6-Pad6) -> /rear_bumper
- J3 pad 7: unconnected-(J2-Pin_7-Pad7) -> /rear_bumper
- J3 pad 8: unconnected-(J2-Pin_8-Pad8) -> /rear_bumper
- U3 pad 12: unconnected-(U1-MTMS/GPIO14/ADC2_CH6-Pad12) -> /imu_drdy
- U3 pad 7: unconnected-(U1-32K_XP/GPIO32/ADC1_CH4-Pad7) -> /front_bumper
- U3 pad 8: unconnected-(U1-32K_XN/GPIO33/ADC1_CH5-Pad8) -> /rear_bumper
Routing:
- net VCC: track 155.7 -> 0.00 mm, vias 1 -> 0
- net /L_ENCODER_A_LV: track 124.0 -> 0.00 mm, vias 1 -> 0
- net /R_ENCODER_A_LV: track 115.4 -> 0.00 mm, vias 1 -> 0
- net +3V3: track 110.9 -> 0.00 mm
- net /R_ENCODER_B_LV: track 93.2 -> 0.00 mm, vias 1 -> 0
- net /L_ENCODER_B_LV: track 85.5 -> 0.00 mm
- net /display_rst: track 84.3 -> 0.00 mm, vias 1 -> 0
- net /ucp_reset_lv: track 84.1 -> 0.00 mm, vias 1 -> 0
- net /display_RS_DC: track 81.6 -> 0.00 mm, vias 1 -> 0
- net /R_MOTOR_PWM: track 80.9 -> 0.00 mm
- net /R_MOTOR_DIR: track 77.9 -> 0.00 mm, vias 1 -> 0
- net /V_BATTERY_MEASUREMENT: track 76.8 -> 0.00 mm
- net /ucp_status_lv: track 76.2 -> 0.00 mm
- net /L_MOTOR_PWM: track 75.0 -> 0.00 mm
- net /ucp_motors_lv: track 73.8 -> 0.00 mm, vias 1 -> 0
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
Commit message: 20251129
Parts:
- added C3: 100nF, Capacitor_THT:C_Axial_L3.8mm_D2.6mm_P7.50mm_Horizontal, F.Cu at (120.8, 73.8)
- added C4: 100nF, Capacitor_THT:C_Axial_L3.8mm_D2.6mm_P7.50mm_Horizontal, F.Cu at (120.8, 83.2)
- added CP1: 100uF/10V, Capacitor_THT:CP_Radial_D5.0mm_P2.50mm, F.Cu at (123.4, 78.5)
- added CP2: 100uF/10V, Capacitor_THT:CP_Radial_D5.0mm_P2.50mm, F.Cu at (123.4, 69.2)
- U4: footprint p3dx:GY_271 -> p3dx:MPU6050
- moved U4 106.0 mm to (61.6, 76.3), turned to 90 degrees
- moved R5 81.8 mm to (146.2, 63.5)
- moved J6 80.2 mm to (145.0, 70.9)
- moved R3 77.7 mm to (119.2, 63.5)
- moved J5 65.7 mm to (132.6, 70.9)
- moved R1 56.4 mm to (98.2, 63.5)
- moved R4 52.3 mm to (71.2, 63.5)
- moved U3 34.1 mm to (98.4, 92.7), turned to -90 degrees
- moved U2 27.3 mm to (139.9, 105.4)
- moved U1 22.3 mm to (96.4, 81.0), turned to 90 degrees
- moved R2 21.0 mm to (71.2, 86.3)
- moved J3 10.0 mm to (155.0, 55.2)
- moved J4 9.11 mm to (57.8, 83.7)
- moved J2 7.74 mm to (127.7, 55.2)
- moved J1 5.14 mm to (80.1, 55.2)
Connections:
- U3 pad 12: /imu_drdy -> /imu_int
- U4 pad 5: /imu_drdy -> unconnected-(U4-XDA-Pad5)
Routing:
- net +3V3: track 0.00 -> 170.2 mm, vias 0 -> 1
- net VCC: track 0.00 -> 143.4 mm, vias 0 -> 1
- net /R_MOTOR_DIR: track 0.00 -> 129.7 mm, vias 0 -> 1
- net /rear_bumper: track 0.00 -> 123.5 mm, vias 0 -> 1
- net /lidar-tx: track 0.00 -> 116.8 mm, vias 0 -> 1
- net /MOTOR_ENABLE: track 0.00 -> 116.5 mm, vias 0 -> 1
- net /lidar-rx: track 0.00 -> 111.1 mm, vias 0 -> 1
- net /ucp_status_lv: track 0.00 -> 95.4 mm, vias 0 -> 2
- net /R_MOTOR_PWM: track 0.00 -> 91.3 mm, vias 0 -> 1
- net /L_MOTOR_PWM: track 0.00 -> 86.2 mm, vias 0 -> 1
- net /L_MOTOR_DIR: track 0.00 -> 83.2 mm, vias 0 -> 1
- net /L_ENCODER_B_LV: track 0.00 -> 81.0 mm, vias 0 -> 1
- net /R_ENCODER_B_LV: track 0.00 -> 77.2 mm, vias 0 -> 1
- net /ucp_motors: track 0.00 -> 72.0 mm, vias 0 -> 1
- net /ucp_status: track 0.00 -> 61.1 mm
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Other:
- board text added: "+5V(red)"
- board text added: "Front Bumpers"
- board text added: "GND(Black)"
- board text added: "Motor Controller"
- board text added: "Pioneer 3DX Mobile Robot Controller Department: ATIx/Mechatronics Design by: Gerard Harkema © 2025"
- board text added: "Power"
- board text added: "Rear Bumpers"
- board text added: "User Panel Control"

Commit message: 20251130
Parts:
- added G***: LOGO, LOGO, F.Cu at (64.8, 124.8)
- added G***: LOGO, LOGO, F.Cu at (91.5, 124.8)
