File: kiCad/P3DX_Controller/P3DX_Controller.kicad_pcb (KiCad board)
At the start: 2 copper layers, 130 x 80 mm, 26 parts, among them J1 Conn_01x10_Pin, J2 Conn_01x26_Pin, J3 Conn_01x10_Pin, J4 Conn_01x16_Pin, J5 Conn_01x03_Pin, J6 Conn_01x05_Pin, U2 TXS0108EPW, U3 ESP32-S3-DevKitC

Commit message: added buzzer
Parts:
- R2: value 10k -> 560k
- R3: value 10k -> 100k
Connections:
- J1 pad 1: /front_bumper -> /rear_bumper
- J1 pad 2: /front_bumper -> /rear_bumper
- J1 pad 3: /front_bumper -> /rear_bumper
- J1 pad 4: /front_bumper -> /rear_bumper
- J1 pad 5: /front_bumper -> /rear_bumper
- J1 pad 6: /front_bumper -> /rear_bumper
- J1 pad 7: /front_bumper -> /rear_bumper
- J1 pad 8: /front_bumper -> /rear_bumper
- J3 pad 1: /rear_bumper -> /front_bumper
- J3 pad 2: /rear_bumper -> /front_bumper
- J3 pad 3: /rear_bumper -> /front_bumper
- J3 pad 4: /rear_bumper -> /front_bumper
- J3 pad 5: /rear_bumper -> /front_bumper
- J3 pad 6: /rear_bumper -> /front_bumper
- J3 pad 7: /rear_bumper -> /front_bumper
- J3 pad 8: /rear_bumper -> /front_bumper
- U3 pad 14: /front_bumper -> /rear_bumper
- U3 pad 30: /rear_bumper -> /front_bumper
Changed lines of the file:
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@@
 			(layers "*.Cu" "*.Mask")
 			(remove_unused_layers no)
-			(net 9 "/front_bumper")
+			(net 28 "/rear_bumper")
 			(pinfunction "GPIO46")
 			(pintype "bidirectional")
@@
 			(layers "*.Cu" "*.Mask")
 			(remove_unused_layers no)
-			(net 28 "/rear_bumper")
+			(net 9 "/front_bumper")
 			(pinfunction "GPIO45")
 			(pintype "bidirectional")
@@
 			(remove_unused_layers no)
 			(roundrect_rratio 0.147059)
-			(net 28 "/rear_bumper")
+			(net 9 "/front_bumper")
 			(pinfunction "Pin_1")
 			(pintype "passive")
@@
 			(layers "*.Cu" "*.Mask")
 			(remove_unused_layers no)
-			(net 28 "/rear_bumper")
+			(net 9 "/front_bumper")
 			(pinfunction "Pin_2")
 			(pintype "passive")
@@
 			(layers "*.Cu" "*.Mask")
 			(remove_unused_layers no)
-			(net 28 "/rear_bumper")
+			(net 9 "/front_bumper")
 			(pinfunction "Pin_3")
 			(pintype "passive")
@@
 			(layers "*.Cu" "*.Mask")
 			(remove_unused_layers no)
-			(net 28 "/rear_bumper")
+			(net 9 "/front_bumper")
 			(pinfunction "Pin_4")
 			(pintype "passive")
@@
 			(layers "*.Cu" "*.Mask")
 			(remove_unused_layers no)
-			(net 28 "/rear_bumper")
+			(net 9 "/front_bumper")
 			(pinfunction "Pin_5")
 			(pintype "passive")
@@
 			(layers "*.Cu" "*.Mask")
 			(remove_unused_layers no)
-			(net 28 "/rear_bumper")
+			(net 9 "/front_bumper")
 			(pinfunction "Pin_6")
 			(pintype "passive")
@@
 			(layers "*.Cu" "*.Mask")
 			(remove_unused_layers no)
-			(net 28 "/rear_bumper")
+			(net 9 "/front_bumper")
 			(pinfunction "Pin_7")
 			(pintype "passive")
@@
 			(layers "*.Cu" "*.Mask")
 			(remove_unused_layers no)
-			(net 28 "/rear_bumper")
+			(net 9 "/front_bumper")
 			(pinfunction "Pin_8")
 			(pintype "passive")
@@
 			)
 		)
-		(property "Value" "10k"
+		(property "Value" "560k"
 			(at 3.81 1.92 0)
 			(layer "F.Fab")
@@
 			)
 		)
-		(property "Value" "10k"
+		(property "Value" "100k"
 			(at 3.81 1.92 0)
 			(layer "F.Fab")
@@
 			(remove_unused_layers no)
 			(roundrect_rratio 0.147059)
-			(net 9 "/front_bumper")
+			(net 28 "/rear_bumper")
 			(pinfunction "Pin_1")
 			(pintype "passive")
@@
 			(layers "*.Cu" "*.Mask")
 			(remove_unused_layers no)
-			(net 9 "/front_bumper")
+			(net 28 "/rear_bumper")
 			(pinfunction "Pin_2")
 			(pintype "passive")
@@
 			(layers "*.Cu" "*.Mask")
 			(remove_unused_layers no)
-			(net 9 "/front_bumper")
+			(net 28 "/rear_bumper")
 			(pinfunction "Pin_3")
 			(pintype "passive")
@@
 			(layers "*.Cu" "*.Mask")
 			(remove_unused_layers no)
-			(net 9 "/front_bumper")
+			(net 28 "/rear_bumper")
 			(pinfunction "Pin_4")
 			(pintype "passive")
@@
 			(layers "*.Cu" "*.Mask")
 			(remove_unused_layers no)
-			(net 9 "/front_bumper")
+			(net 28 "/rear_bumper")
 			(pinfunction "Pin_5")
 			(pintype "passive")
@@
 			(layers "*.Cu" "*.Mask")
 			(remove_unused_layers no)
-			(net 9 "/front_bumper")
+			(net 28 "/rear_bumper")
 			(pinfunction "Pin_6")
 			(pintype "passive")
@@
 			(layers "*.Cu" "*.Mask")
 			(remove_unused_layers no)
-			(net 9 "/front_bumper")
+			(net 28 "/rear_bumper")
 			(pinfunction "Pin_7")
 			(pintype "passive")
@@
 			(layers "*.Cu" "*.Mask")
 			(remove_unused_layers no)
-			(net 9 "/front_bumper")
+			(net 28 "/rear_bumper")
 			(pinfunction "Pin_8")
 			(pintype "passive")
